File: Hardware/_autosave-Flight Controller.kicad_pcb (KiCad board)
At the start: 6 copper layers, 164 parts, among them J1 USB4110GFA, J2 ST_LINK, J3 4in1 ESC, J4 FPV, J5 GPS, J6 RC Receiver, SW1 reset, SW2 SSSS810701, U1 TPS54302, U10 W25Q128JVSIQ, U11 STM32H743VITx, U12 BMI270, U2 AP63205WU, U3 AZ1117-3.3, U4 USBLC6-2SC6, U5 AT7456E, U6 INA226, U7 ICM-42688-P, U8 QMC5883P, U9 BMP388, Y1 27Mhz 20pF, Y2 8MHz 12pF

Commit message: This commit completes the Schematics
Parts:
- added TP13: servos, Solderpoint:Solderpad, F.Cu at (71.6, 17.5)
- added TP16: servos, Solderpoint:Solderpad, F.Cu at (73.6, 17.5)
- added TP19: servos, Solderpoint:Solderpad, F.Cu at (75.6, 17.5)
- added TP7: servos, Solderpoint:Solderpad, F.Cu at (69.6, 17.5)
- H1, H2, H3, H4: footprint MountingHole:MountingHole_2.2mm_M2_Pad_Via -> MountingHole:MountingHole_3.2mm_M3_Pad_Via
- R19: value R_Shunt -> FRM252WFR020TN; footprint Resistor_SMD:R_2512_6332Metric_Pad1.40x3.35mm_HandSolder -> memo:R2512
- moved TP1 87.8 mm to (27.8, 95.7)
- moved TP10 87.8 mm to (27.8, 98.8)
- moved TP11 87.8 mm to (29.8, 98.8)
- moved TP12 87.8 mm to (31.8, 98.8)
- moved TP14 87.8 mm to (33.8, 98.8)
- moved TP15 87.8 mm to (35.8, 98.8)
- moved TP17 87.8 mm to (37.8, 98.8)
- moved TP18 87.8 mm to (39.8, 98.8)
- moved TP2 87.8 mm to (29.8, 95.7)
- moved TP20 87.8 mm to (41.8, 98.8)
- moved TP21 87.8 mm to (27.8, 102.0)
- moved TP22 87.8 mm to (29.8, 102.0)
- moved TP23 87.8 mm to (31.8, 102.0)
- moved TP24 87.8 mm to (33.8, 102.0)
- moved TP25 87.8 mm to (35.8, 102.0)
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- renumbered TP9 to TP10, TP10 to TP11, TP11 to TP12, TP12 to TP14, TP13 to TP15, TP14 to TP17, TP15 to TP18, TP16 to TP20, TP17 to TP21, TP18 to TP22, TP19 to TP23, TP20 to TP24, TP21 to TP25, TP22 to TP26, TP23 to TP27, TP24 to TP28, TP25 to TP29, TP26 to TP30, TP27 to TP31, TP28 to TP32, TP29 to TP33, TP30 to TP34, TP31 to TP35, TP32 to TP36, TP33 to TP37, TP34 to TP38, TP35 to TP39, TP36 to TP40, TP37 to TP41, TP7 to TP8, TP8 to TP9
Connections:
- R17 pad 2: Net-(R17-Pad2) -> VBAT_Sense
- R18 pad 2: Net-(R18-Pad2) -> VBAT_MEASURE
- R19 pad 1: VBAT_MEASURE -> VBAT_Sense
- R19 pad 2: Net-(R18-Pad2) -> VBAT_MEASURE
- U11 pad 77: Servo_4 -> SERVO_4
Other:
- board outline added: 69.4 x 71.1 mm
