File: Hardware/Flight Controller.kicad_sch (KiCad schematic)
At the start: 146 parts, among them J1 USB4110GFA, J2 ST_LINK, J3 RC Receiver, SW1 reset, SW2 SSSS810701, U1 TPS54302, U10 W25Q128JVSIQ, U11 STM32H743VITx, U12 ICM-42688-P, U2 TPS54302, U3 AZ1117-3.3, U4 USBLC6-2SC6, U5 INA226, U6 AT7456E, U7 ICM-42688-P, U8 QMC5883P, U9 BMP388, Y1 27Mhz 20pF, Y2 8MHz 12pF

Commit message: Changed 5V Regulator, pin mapping for ESC and motors
Parts:
- removed C11, C14: 22uF, Capacitor_SMD:C_0603_1608Metric, symbol Device:C_Small
- removed C16: 75pF, Capacitor_SMD:C_0603_1608Metric, symbol Device:C_Small
- removed C2: 10uF, Capacitor_SMD:C_0603_1608Metric, symbol Device:C_Small
- removed C4, C45, C9: 0.1uF, Capacitor_SMD:C_0603_1608Metric, symbol Device:C_Small
- removed C48: 2.2uF, Capacitor_SMD:C_0603_1608Metric, symbol Device:C_Small
- removed C52: 10nF, Capacitor_SMD:C_0603_1608Metric, symbol Device:C_Small
- removed L2: 15uH, Inductor_SMD:L_TracoPower_TCK-047_5.2x5.8mm, symbol Device:L_Iron
- removed L3: 10uH, Inductor_SMD:L_TracoPower_TCK-047_5.2x5.8mm, symbol Device:L_Iron
- removed R10: 100k, Resistor_SMD:R_0402_1005Metric, symbol Device:R_Small
- removed R11: 13.3k, Resistor_SMD:R_0402_1005Metric, symbol Device:R_Small
- removed R20: 10k, Resistor_SMD:R_0402_1005Metric, symbol Device:R_Small
- removed R23: 1k, Resistor_SMD:R_0402_1005Metric, symbol Device:R_Small
- removed R34: 0, Resistor_SMD:R_0402_1005Metric, symbol Device:R_Small
- removed R9: 49.9, Resistor_SMD:R_0402_1005Metric, symbol Device:R_Small
- removed TP3: Motor_5, Solderpoint:Solderpad, symbol Connector:TestPoint
- removed U12: ICM-42688-P, memo:PQFN50P300X250X97-14N, symbol ICM-42688:ICM-42688-P
- removed U2: TPS54302, Package_TO_SOT_SMD:SOT-23-6, symbol Regulator_Switching:TPS54302
- added C13, C3, C40, C41, C46, C8: 0.1uF, Capacitor_SMD:C_0603_1608Metric, symbol Device:C_Small
- added D3, D4, D5, D6: LED, symbol Device:LED
- added H1, H2, H3, H4: MountingHole, MountingHole:MountingHole_2.2mm_M2_Pad_Via, symbol Mechanical:MountingHole
- added J3: 4in1 ESC, Connector_JST:JST_SH_SM08B-SRSS-TB_1x08-1MP_P1.00mm_Horizontal, symbol Connector_Generic:Conn_01x08
- added J4: FPV, Connector_JST:JST_SH_SM04B-SRSS-TB_1x04-1MP_P1.00mm_Horizontal, symbol Connector_Generic:Conn_01x04
- added J5: GPS, Connector_JST:JST_SH_SM06B-SRSS-TB_1x06-1MP_P1.00mm_Horizontal, symbol Connector_Generic:Conn_01x06
- added L2: 15uH, symbol Device:L_Small
- added L3: 4.7uH, symbol Device:L_Small
- added R29, R30, R31: 330, Resistor_SMD:R_0402_1005Metric, symbol Device:R_Small
- added TP13, TP17, TP22, TP27, TP35, TP37: GND, Solderpoint:Solderpad, symbol Connector:TestPoint
- added TP20, TP29: VIDEO_OUT, Solderpoint:Solderpad, symbol Connector:TestPoint
- added TP25: VTX_TX, Solderpoint:Solderpad, symbol Connector:TestPoint
- added TP26: TELEMETRY_RX, Solderpoint:Solderpad, symbol Connector:TestPoint
- added TP31: TELEMETRY_TX, Solderpoint:Solderpad, symbol Connector:TestPoint
- added TP32, TP34: 5V, Solderpoint:Solderpad, symbol Connector:TestPoint
- added TP36: PWR, Solderpoint:Solderpad, symbol Connector:TestPoint
- added U12: BMI270, memo:XDCR_BMI270, symbol bmi270:BMI270
- added U2: AP63205WU, Package_TO_SOT_SMD:TSOT-23-6, symbol Regulator_Switching:AP63205WU
- C42: renamed from C44; footprint Capacitor_SMD:C_0603_1608Metric -> Capacitor_SMD:C_0402_1005Metric
- C44: renamed from C47; footprint Capacitor_SMD:C_0603_1608Metric -> Capacitor_SMD:C_0402_1005Metric
- C45: renamed from C46; value 14pF -> 27pF; footprint Capacitor_SMD:C_0603_1608Metric -> Capacitor_SMD:C_0402_1005Metric
- C47: renamed from C49; footprint Capacitor_SMD:C_0603_1608Metric -> Capacitor_SMD:C_0402_1005Metric
- C49: renamed from C53; footprint Capacitor_SMD:C_0603_1608Metric -> Capacitor_SMD:C_0402_1005Metric
- C51: renamed from C56; footprint Capacitor_SMD:C_0603_1608Metric -> Capacitor_SMD:C_0402_1005Metric
- C52: renamed from C55; value 14pF -> 27pF; footprint Capacitor_SMD:C_0603_1608Metric -> Capacitor_SMD:C_0402_1005Metric
- C53: renamed from C54; footprint Capacitor_SMD:C_0603_1608Metric -> Capacitor_SMD:C_0402_1005Metric
- C54: renamed from C57; footprint Capacitor_SMD:C_0603_1608Metric -> Capacitor_SMD:C_0402_1005Metric
- R17: renamed from R21; value 10 -> 7.5
- R18: renamed from R22; value 10 -> 7.5
- R19: renamed from R24; footprint Resistor_SMD:R_Shunt_Vishay_WSR2_WSR3_KelvinConnection -> Resistor_SMD:R_2512_6332Metric_Pad1.40x3.35mm_HandSolder
- R5: value 511k -> 330
- R6: value 105k -> 1k
- TP7: value GND -> 5V
- renumbered C12 to C10, C13 to C11, C15 to C12, C17 to C14, C18 to C15, C19 to C16, C20 to C17, C21 to C18, C22 to C19, C3 to C2, C23 to C20, C24 to C21, C26 to C22, C25 to C23, C27 to C24, C28 to C25, C29 to C26, C30 to C27, C31 to C28, C32 to C29, C33 to C30, C34 to C31, C35 to C32, C36 to C33, C37 to C34, C38 to C35, C39 to C36, C40 to C37, C41 to C38, C42 to C39, C5 to C4, C50 to C48, C6 to C5, C51 to C50, C7 to C6, C8 to C7, C10 to C9, J3 to J6, R13 to R10, R14 to R11, R15 to R12, R16 to R13, R17 to R14, R18 to R15, R19 to R16, R25 to R20, R26 to R21, R27 to R22, R28 to R23, R29 to R24, R30 to R25, R31 to R26, R32 to R27, R33 to R28, R35 to R32, R36 to R33, R37 to R34, R12 to R9, TP15 to TP14, TP14 to TP15, TP17 to TP18, TP18 to TP19, TP19 to TP21, TP20 to TP23, TP21 to TP24, TP22 to TP28, TP4 to TP3, TP23 to TP30, TP24 to TP33, TP5 to TP4, TP8 to TP5, TP13 to TP8, U6 to U5, U5 to U6
Connections:
- net BMP_SCL is gone; now on net I2C2_SCL: R21.2
- net BMP_SDA is gone; now on net I2C2_SDA: R23.2
- net +3.3V: now also R5.2, C40.1, U12.5 (VDDIO)
- net +3.3VA: now also C46.1, U12.8 (VDD)
- net +5V: now also R6.2, C13.2, J4.1 (Pin_1), J5.1 (Pin_1), L3.2, TP32.1, TP34.1, U2.1 (FB)
- net +pwr_out: now also TP7.1, L2.2, TP36.1
- net GND: now also C13.1, C3.1, C40.2, C41.1, C46.2, D3.1 (K), D4.1 (K), D5.1 (K), D6.1 (K), J3.2 (Pin_2), J4.4 (Pin_4), J5.6 (Pin_6), TP13.1, TP22.1, TP27.1, TP35.1, TP37.1, U12.6 (GNDIO), U12.7 (GND), U2.4 (GND); no longer R6.2, TP7.1
- net GPS_RX: now also J5.3 (Pin_3)
- net GPS_SCL: now also J5.5 (Pin_5)
- net GPS_SDA: now also J5.4 (Pin_4)
- net GPS_TX: now also J5.2 (Pin_2)
- net IMU2_CS: now also U12.12 (CSB)
- net IMU2_INT1: now also U12.4 (INT1)
- net IMU2_MISO: now also U12.1 (SDO)
- net IMU2_MOSI: now also U12.14 (SDX)
- net IMU2_SCLK: now also U12.13 (SCX)
- net STATUS_LED_1: now also R30.2
- net STATUS_LED_2: now also R29.2
- net TELEMETRY_RX: now also TP26.1
- net TELEMETRY_TX: now also TP31.1
- net VBAT: now also J3.1 (Pin_1), TP17.1
- net VBAT_MEASURE: now also C3.2, U2.2 (EN), U2.3 (IN); no longer R5.1
- net VIDEO_IN: now also J4.2 (Pin_2), TP20.1
- net VIDEO_OUT: now also TP29.1
- net at C7.2, U1.2 (SW): now also L2.1
- net at R17.1, U6.10 (Vin+): now also C22.1
- net at R17.2, R19.3: no longer C22.1
- net at R18.2, R19.2: no longer C22.2
- net ESC_RX: now reaches U11.37 (PE7)
- net ESC_RX: now also J3.8 (Pin_8)
- net at U11.52 (PB13): now also R31.1
- net VTX_TX: now reaches U11.98 (PE1)
- net VTX_TX: now also TP25.1
- net at R18.1, U6.9 (Vin-): now also C22.2
- net ADC_VOLTAGE: no longer names the net of U11.17 (PC2_C)
- net EN_5V: no longer names the net of R6.1
- net EN_5V: now also D4.2 (A); no longer R5.2
- net LED_STRIPS: no longer names the net of U11.35 (PB1)
- net T1_CH1 renamed M5
- net M5: now also J3.3 (Pin_3)
- net T1_CH2 renamed M6
- net M6: now also J3.4 (Pin_4)
- net T1_CH3 renamed M7
- net M7: now also J3.5 (Pin_5)
- net T1_CH4 renamed M8
- net M8: now also J3.6 (Pin_6)
- net T2_CH1 renamed Servo_4
- new net: D3.2 (A), R5.1
- new net: C8.1, L3.1, U2.5 (SW)
- new net: C8.2, U2.6 (BST)
- new net: D6.2 (A), R30.1
- new net: D5.2 (A), R29.1
- new net CC: C41.2, J4.3 (Pin_3), R31.2
- no-connect marks 58 -> 60
Other:
- note added: "14.8"
- note added: "2*(20 - 5) = 30pF"
- note added: "FPV 9/12V"
- note added: "Telemetry"
- note added: "VTX"
- note removed: "2*(12 - 5) = 14pF"
- note removed: "FB pin max = 7V, V_out = V_in * (R2 / (R1 + R2)) V_out = 1.7V"
- note removed: "voltage sensor"
- moved on the sheet: C15, C17, C19, C20, C21, C22, C23, C25, C26, C43, C45, C48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

Commit message: This commit completes the Schematics
Parts:
- removed R19: R_Shunt, Resistor_SMD:R_2512_6332Metric_Pad1.40x3.35mm_HandSolder, symbol Device:R_Shunt
- added R19: FRM252WFR020TN, memo:R2512, symbol shunt:FRM252WFR020TN
- added TP13, TP16, TP19, TP7: servos, Solderpoint:Solderpad, symbol Connector:TestPoint
- D3, D4, D5, D6: footprint (none) -> LED_SMD:LED_0402_1005Metric
- H1, H2, H3, H4: footprint MountingHole:MountingHole_2.2mm_M2_Pad_Via -> MountingHole:MountingHole_3.2mm_M3_Pad_Via
- L2, L3: footprint (none) -> Inductor_SMD:L_TracoPower_TCK-047_5.2x5.8mm
- renumbered TP9 to TP10, TP10 to TP11, TP11 to TP12, TP12 to TP14, TP13 to TP15, TP14 to TP17, TP15 to TP18, TP16 to TP20, TP17 to TP21, TP18 to TP22, TP19 to TP23, TP20 to TP24, TP21 to TP25, TP22 to TP26, TP23 to TP27, TP24 to TP28, TP25 to TP29, TP26 to TP30, TP27 to TP31, TP28 to TP32, TP29 to TP33, TP30 to TP34, TP31 to TP35, TP32 to TP36, TP33 to TP37, TP34 to TP38, TP35 to TP39, TP36 to TP40, TP37 to TP41, TP7 to TP8, TP8 to TP9
Connections:
- net SERVO_1: now also TP7.1
- net SERVO_2: now also TP13.1
- net SERVO_3: now also TP16.1
- net VBAT_MEASURE: now also R18.2, R19.2
- net VBAT_Sense: now also R17.2, R19.1
- net Servo_4 renamed SERVO_4
- net SERVO_4: now also TP19.1

Commit message: This commit changes Battery Filtering and Fixes Magnetometer wiring
Parts:
- removed L1: 10uH, Inductor_SMD:L_TracoPower_TCK-047_5.2x5.8mm, symbol Device:L_Iron
- added Q1: AO3407A, memo:AO3407A, symbol AO3407A:AO3407A
- added R5: 0, Resistor_SMD:R_0402_1005Metric, symbol Device:R_Small
- C27: footprint Capacitor_SMD:C_0603_1608Metric -> Capacitor_SMD:C_0805_2012Metric
- C28, C31, C35: footprint Capacitor_SMD:C_0603_1608Metric -> Capacitor_SMD:C_0402_1005Metric
- L1: renamed from L2; footprint Inductor_SMD:L_TracoPower_TCK-047_5.2x5.8mm -> memo:IND-SMD_L5.4-W5.2
- L2: renamed from L3; footprint Inductor_SMD:L_TracoPower_TCK-047_5.2x5.8mm -> memo:IND-SMD_L4.4-W4.2
- renumbered C5 to C4, C4 to C5, C7 to C6, C6 to C7, R9 to R10, R10 to R11, R11 to R12, R12 to R13, R13 to R14, R14 to R15, R15 to R16, R16 to R17, R17 to R18, R18 to R19, R19 to R20, R20 to R21, R21 to R22, R22 to R23, R23 to R24, R24 to R25, R25 to R26, R26 to R27, R27 to R28, R28 to R29, R29 to R30, R30 to R31, R31 to R32, R32 to R33, R33 to R34, R34 to R35, R5 to R6, R6 to R7, R7 to R8, R8 to R9
Connections:
- net +3.3V: now also C28.1, U8.2 (VDD)
- net GND: now also R5.1
- net VBAT: now also Q1.3 (D)
- net VBAT_Filtered: now also Q1.2 (S)
- net IN+: now reaches C22.1, R18.1, U6.10 (Vin+)
- net A1: now reaches R13.2, U6.1 (A1)
- net A0: now reaches R14.2, U6.2 (A0)
- net IN-: now reaches C22.2, R19.1, U6.9 (Vin-)
- new net: Q1.1 (G), R5.2
Other:
- note added: "TVS and reverse polarity protection"
- note removed: "LC filter and TVS protection"
- moved on the sheet: C5, C7

Commit message: This commits adds latest Schematics
Parts:
- added C14: 22uF, Capacitor_SMD:C_0603_1608Metric, symbol Device:C_Small
- C13: value 0.1uF -> 22uF
- C3: value 0.1uF -> 10uF
- C30: renamed from C29; footprint Capacitor_SMD:C_0603_1608Metric -> Capacitor_SMD:C_0402_1005Metric
- C33: renamed from C32; footprint Capacitor_SMD:C_0603_1608Metric -> Capacitor_SMD:C_0402_1005Metric
- renumbered C14 to C15, C15 to C16, C16 to C17, C17 to C18, C18 to C19, C19 to C20, C20 to C21, C21 to C22, C22 to C23, C23 to C24, C24 to C25, C25 to C26, C26 to C27, C27 to C28, C28 to C29, C30 to C31, C31 to C32, C33 to C34, C34 to C35, C35 to C36, C36 to C37, C37 to C38, C38 to C39, C39 to C40, C40 to C41, C41 to C42, C42 to C43, C43 to C44, C44 to C45, C45 to C46, C46 to C47, C47 to C48, C48 to C49, C49 to C50, C50 to C51, C51 to C52, C52 to C53, C53 to C54, C54 to C55
Connections:
- net +5V: now also C14.2
- net GND: now also C14.1
- net reset: now also R28.2, U10.7 (/HOLD/RESET(IO3))
- net 5V_SW: now reaches C8.1, L2.1, U2.5 (SW)
- net bst: now reaches C8.2, U2.6 (BST)
- net SW: now reaches C6.2, L1.1, U1.2 (SW)
- net boot: now reaches C6.1, U1.6 (BOOT)
- net c: now reaches C31.1, U8.10 (C1), U8.11 (GND), U8.9 (GND)
- net wp: now reaches R27.1, U10.3 (/WP(IO2))
Other:
- moved on the sheet: R8
