File: Hardware/Flight Controller.kicad_sch (KiCad schematic)
At the start: 0 parts

Commit message: Added Necessary Connectors, pads and comments in the respective file
Other:
- note added: "Signal Bidirectional"
- note added: "TVS + reverse polarity protection Dual buck converters (5 V + 9/12 V) Dual LDO rails (3.3V digital + 3.3V IMU) USB-C power + automatic power switching Basic input filtering INA226 voltage/current monitor - I²C"
- note removed: "Signal"
- note removed: "TVS + reverse polarity protection Dual buck converters (5 V + 9/12 V) Dual LDO rails (3.3 V digital + 3.3 V sensors) USB-C power + automatic power switching Basic input filtering INA226 voltage/current monitor - I²"
Changed lines of the file:
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@@
 		)
 	)
-	(text "Signal"
+	(text "Signal Bidirectional"
 		(exclude_from_sim no)
 		(at 589.788 78.867 0)
@@
 		)
 	)
-	(text "TVS + reverse polarity protection\n\nDual buck converters (5 V + 9/12 V)\n\nDual LDO rails (3.3 V digital + 3.3 V sensors)\n\nUSB-C power + automatic power switching\n\nBasic input filtering\n\nINA226 voltage/current monitor - I²"
+	(text "TVS + reverse polarity protection\n\nDual buck converters (5 V + 9/12 V)\n\nDual LDO rails (3.3V digital + 3.3V IMU)\n\nUSB-C power + automatic power switching\n\nBasic input filtering\n\nINA226 voltage/current monitor - I²C"
 		(exclude_from_sim no)
 		(at 94.742 91.44 0)
@@
 				(thickness 0.4064)
 				(bold yes)
-				(color 255 15 7 1)
-			)
+				(color 194 0 0 1)
+			)
+		)
+	)
+	(polyline
+		(pts
+			(xy 135.255 42.545) (xy 135.255 29.845)
+		)
+		(stroke
+			(width 1.27)
+			(type default)
+			(color 194 0 0 1)
+		)
+	)
+	(polyline
+		(pts
+			(xy 343.535 153.67) (xy 415.925 153.67)
+		)
+		(stroke
+			(width 1.27)
+			(type solid)
 		)
 	)
@@
 			(width 0.762)
 			(type default)
-			(color 255 4 10 1)
+			(color 194 0 0 1)
+		)
+	)
+	(polyline
+		(pts
+			(xy 463.55 231.775) (xy 463.55 288.925)
+		)
+		(stroke
+			(width 1.27)
+			(type default)
+		)
+	)
+	(polyline
+		(pts
+			(xy 269.24 29.845) (xy 269.24 57.785)
+		)
+		(stroke
+			(width 1.27)
+			(type default)
+			(color 194 0 0 1)
+		)
+	)
+	(polyline
+		(pts
+			(xy 132.715 161.925) (xy 132.715 182.245)
+		)
+		(stroke
+			(width 1.27)
+			(type solid)
+			(color 194 0 0 1)
+		)
+	)
+	(polyline
+		(pts
+			(xy 150.495 288.925) (xy 463.55 288.925)
+		)
+		(stroke
+			(width 1.27)
+			(type default)
+		)
+	)
+	(polyline
+		(pts
+			(xy 149.86 210.82) (xy 201.295 210.82)
+		)
+		(stroke
+			(width 1.27)
+			(type default)
 		)
 	)
@@
 			(width 0.762)
 			(type default)
+		)
+	)
+	(polyline
+		(pts
+			(xy 135.255 29.845) (xy 453.39 29.845)
+		)
+		(stroke
+			(width 1.27)
+			(type default)
+			(color 194 0 0 1)
+		)
+	)
+	(polyline
+		(pts
+			(xy 453.39 29.845) (xy 453.39 75.565)
+		)
+		(stroke
+			(width 1.27)
+			(type default)
+			(color 194 0 0 1)
 		)
 	)
@@
 		(fields_autoplaced yes)
 		(stroke
-			(width 0.1524)
+			(width 1.27)
 			(type solid)
 		)
@@
 		(fields_autoplaced yes)
 		(stroke
-			(width 0.1524)
+			(width 1.27)
 			(type solid)
 		)
@@
 		(dnp no)
 		(stroke
-			(width 0.1524)
+			(width 1.27)
 			(type solid)
 		)
@@
 		(dnp no)
 		(stroke
-			(width 0.1524)
+			(width 1.27)
 			(type solid)
 		)
@@
 		)
 		(property "Sheetname" "Sensors and Peripherals"
-			(at 39.243 182.245 0)
-			(effects
-				(font
+			(at 48.768 180.848 0)
+			(effects
+				(font

Commit message: Added Digital Airspeed Sensor Connector, Changed the Magnetometer
Other:
- note added: "ICM-42688P (primary IMU) - SPI BMI270 (backup IMU) - SPI BMP388 barometer - I²C Magnetometer (LIS3MDL) - I²C AT7456E OSD - SPI W25Q128 flash memory (16 Mbit) - SPI CAN transceiver (SN65HVD230) - FDCAN"
- note removed: "Airspeed and mag, yet to be picked"
- note removed: "ICM-42688P (primary IMU) - SPI BMI270 (backup IMU) - SPI BMP388 barometer - I²C Magnetometer (IST8310 / LIS3MDL) - I²C Airspeed sensor (MS4525DO) - I²C AT7456E OSD - SPI W25Q128 flash memory (16 Mbit) - SPI CAN transceiver (SN65HVD230) - FDCAN"
Changed lines of the file:
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@@
 		(end 680.72 207.01)
 		(stroke
-			(width 0.762)
+			(width 1.27)
 			(type dash)
 		)
@@
 		)
 	)
-	(text "Airspeed and mag, yet to be picked"
-		(exclude_from_sim no)
-		(at 100.965 285.75 0)
-		(effects
-			(font
-				(size 2.54 2.54)
-				(thickness 0.508)
-				(bold yes)
-				(color 255 0 0 1)
-			)
-		)
-	)
 	(text "Flight Controller Design"
 		(exclude_from_sim no)
@@
 		)
 	)
-	(text "ICM-42688P (primary IMU) - SPI\n\nBMI270 (backup IMU) - SPI\n\nBMP388 barometer - I²C\n\nMagnetometer (IST8310 / LIS3MDL) - I²C\n\nAirspeed sensor (MS4525DO) - I²C\n\nAT7456E OSD - SPI\n\nW25Q128 flash memory (16 Mbit) - SPI\n\nCAN transceiver (SN65HVD230) - FDCAN\n"
+	(text "ICM-42688P (primary IMU) - SPI\n\nBMI270 (backup IMU) - SPI\n\nBMP388 barometer - I²C\n\nMagnetometer (LIS3MDL) - I²C\n\n\nAT7456E OSD - SPI\n\nW25Q128 flash memory (16 Mbit) - SPI\n\nCAN transceiver (SN65HVD230) - FDCAN\n"
 		(exclude_from_sim no)
 		(at 97.917 241.554 0)
@@
 	(polyline
 		(pts
-			(xy 269.24 29.845) (xy 269.24 57.785)
+			(xy 269.24 29.845) (xy 269.24 60.325)
 		)
 		(stroke
@@
 	(polyline
 		(pts
-			(xy 453.39 29.845) (xy 453.39 75.565)
-		)
-		(stroke
+			(xy 453.39 29.845) (xy 453.39 79.375)
+		)
+		(stroke
