File: Hardware/Flight Controller.kicad_sch (KiCad schematic)
At the start: 0 parts

Commit message: added CAN connector
Changed lines of the file:
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@@
 			(font
 				(size 2.54 2.54)
-				(thickness 0.762)
+				(thickness 0.508)
 				(bold yes)
 				(color 0 0 0 1)
@@
 			(font
 				(size 2.54 2.54)
-				(thickness 0.762)
+				(thickness 0.508)
 				(bold yes)
 				(color 0 0 0 1)
@@
 			(font
 				(size 2.54 2.54)
-				(thickness 0.762)
+				(thickness 0.508)
 				(bold yes)
 				(color 0 0 0 1)
