File: Hardware/power.kicad_sch (KiCad schematic)
At the start: 48 parts, among them J1 USB4110GFA, Q1 AO3407A, U1 TPS54302, U2 USBLC6-2SC6, U3 INA226, U4 AP63205WU, U5 AP2112K-3.3, U6 AP7343-33W5-7

Commit message: /HARDWARE: Updated BOM do not Include list
Parts:
- R12: now in the parts list
Changed lines of the file:
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@@
 		(body_style 1)
 		(exclude_from_sim yes)
-		(in_bom no)
+		(in_bom yes)
 		(on_board no)
 		(in_pos_files yes)

Commit message: /HARDWARE: corrected schematics naming
Parts:
- C19: value 4,7uF -> 4.7uF
Changed lines of the file:
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@@
 			)
 		)
-		(property "Value" "4,7uF"
+		(property "Value" "4.7uF"
 			(at 405.13 80.0162 0)
 			(show_name no)
