File: Hardware/Flight Controller.kicad_pcb (KiCad board)
At the start: 6 copper layers, 47.5 x 47.5 mm, 160 parts, among them J1 USB4110GFA, J10 CAN BUS, J2 FPV, J3 ST_LINK, J4 GPS, J5 Airspeed sensor, J6 4in1 ESC, J7 RC Receiver, J8 VTX, J9 DJI, Q1 AO3407A, SW1 reset, SW2 MCU_BOOT, U1 TPS54302, U10 BMI270, U12 BMP388, U13 AT7456E, U14 SN65HVD230, U2 USBLC6-2SC6, U3 INA226, U4 AP63205WU, U5 AP2112K-3.3, U6 AP7343-33W5-7, U7 STM32H743VITx, U8 ICM-42688-P, U9 W25Q128JVSIQ, Y1 ASE-8.000MHZ-LC-T, Y2 27Mhz 20pF, Y3 ASE-27.000MHZ-LC-T

Commit message: changed hella stuff in firmware plan and hardware pcb layout
Parts:
- removed C11, C12: 0.1uF, Capacitor_SMD:C_0603_1608Metric
- removed C13: 10uF, Capacitor_SMD:C_0805_2012Metric
- removed the C21 at (59.7, 101.4)
- removed the C21 at (73.0, 100.1)
- removed D2, D3: PMEG3020EH, Diode_SMD:D_SOD-123F
- removed R10, R11: 7.5, Resistor_SMD:R_0402_1005Metric
- removed R12: FRM252WFR020TN, memo:R2512
- removed R8, R9: 10k, Resistor_SMD:R_0402_1005Metric
- removed U3: INA226, Package_SO:VSSOP-10_3x3mm_P0.5mm
- removed Y3: ASE-27.000MHZ-LC-T, Oscillator:Oscillator_SMD_Abracon_ASE-4Pin_3.2x2.5mm
- added C21: 10nF, Capacitor_SMD:C_0603_1608Metric, F.Cu at (120.7, 92.3)
- added C56: 0.1uF, Capacitor_SMD:C_0402_1005Metric, B.Cu at (141.8, 106.6)
- added J11: CAN BUS, memo:CONN-SMD_4P-P1.00_SM04B-SRSS-TB-LF-SN, B.Cu at (150.7, 100.7)
- added R29: 10k, Resistor_SMD:R_0402_1005Metric, F.Cu at (136.0, 106.1)
- added R30: 10k, Resistor_SMD:R_0402_1005Metric, F.Cu at (137.0, 106.1)
- added TP33: power, Solderpoint:Solderpad, F.Cu at (113.7, 96.3)
- added TP34: power, Solderpoint:Solderpad, F.Cu at (113.7, 98.1)
- added TP35: power, Solderpoint:Solderpad, F.Cu at (135.8, 77.7)
- added TP36: power, Solderpoint:Solderpad, F.Cu at (134.1, 77.7)
- C17, C19, U5: moved to F.Cu
- C18, C20, C55, D8, R20, R21, R22, R27, U6, U9: moved to B.Cu
- C37: footprint Capacitor_SMD:C_0603_1608Metric -> Capacitor_SMD:C_0402_1005Metric; moved to B.Cu
- C43, C44, C51, C52, C53, C54: footprint Capacitor_SMD:C_0603_1608Metric -> Capacitor_SMD:C_0402_1005Metric
- D5, D6, D7: footprint LED_SMD:LED_0402_1005Metric -> LED_SMD:LED_0805_2012Metric
- R6: value 0 -> 1k
- R7: value 0 -> 10k
- moved TP13 117.2 mm to (140.3, 115.6)
- moved TP3 117.0 mm to (142.3, 115.6)
- moved TP5 114.5 mm to (144.2, 115.6)
- moved TP2 113.8 mm to (145.4, 77.8)
- moved TP7 112.6 mm to (141.9, 79.8), turned to 180 degrees
- moved TP16 111.0 mm to (138.4, 115.5)
- moved TP20 110.4 mm to (134.2, 115.6)
- moved TP22 105.9 mm to (140.0, 77.8)
- moved TP24 105.9 mm to (136.3, 115.5)
- moved TP27 102.8 mm to (132.2, 77.7)
- moved TP12 102.8 mm to (143.7, 77.8)
- moved C50 102.3 mm to (137.8, 109.7), turned to -90 degrees
- moved TP29 101.6 mm to (130.6, 115.6)
- moved TP30 101.1 mm to (132.3, 115.6)
- moved C46 100.6 mm to (134.3, 109.1), turned to 90 degrees
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Connections:
- C1 pad 1: VBAT_MEASURE -> VBAT_Filtered
- C10 pad 2: VBAT_MEASURE -> VBAT_Filtered
- C15 pad 2: +5V_REG -> +5V
- C16 pad 2: +5V_REG -> +5V
- C2 pad 1: VBAT_MEASURE -> VBAT_Filtered
- C44 pad 1: +3.3VA -> +3V3_Sensors
- J2 pad 1: +5V -> +pwr_out
- J6 pad 3: M8 -> unconnected-(J6-Pin_3-Pad3)
- J6 pad 4: M7 -> CURR
- J6 pad 5: M6 -> M8
- J6 pad 6: M5 -> M7
- J6 pad 7: unconnected-(J6-Pin_7-Pad7) -> M6
- J6 pad 8: ESC_RX -> M5
- L2 pad 2: +5V_REG -> +5V
- R6 pad 1: GND -> Net-(C56-Pad2)
- R6 pad 2: /Power/A1 -> Net-(U7-PC1)
- R7 pad 1: GND -> Net-(U7-PC1)
- R7 pad 2: /Power/A0 -> VBAT
- TP14 pad 1: VBAT -> +VABT
- U1 pad 3: VBAT_MEASURE -> VBAT_Filtered
- U10 pad 8: +3.3VA -> +3V3_Sensors
- U4 pad 1: +5V_REG -> +5V
- U4 pad 2: VBAT_MEASURE -> VBAT_Filtered
- U4 pad 3: VBAT_MEASURE -> VBAT_Filtered
- U7 pad 15: INA226_ALERT -> unconnected-(U7-PC0-Pad15)
- U7 pad 16: unconnected-(U7-PC1-Pad16) -> Net-(U7-PC1)
- U7 pad 18: unconnected-(U7-PC3_C-Pad18) -> CURR
- U7 pad 51: ESC_RX -> EXPANSION_RX
- U7 pad 52: unconnected-(U7-PB13-Pad52) -> EXPANSION_TX
Routing:
- net unconnected-(U13-NC-Pad27): track 0.00 -> 0.72 mm
Other:
- board size 47.5 x 47.5 mm -> 40.6 x 40.5 mm
- board text added: "3V3"
- board text added: "5V"
- board text added: "BOOT"
- board text added: "CAN_H"
- board text added: "CAN_L"
- board text added: "CLK"
- board text added: "CURR"
- board text added: "DIO"
- board text added: "DJI_RX"
- board text added: "DJI_TX"
- board text added: "GND"
- board text added: "M5"
- board text added: "M6"
- board text added: "M7"
- board text added: "M8"
- board text added: "RESET"
- board text added: "RX"
- board text added: "SBUS"
- board text added: "SCL"
- board text added: "SDA"
- board text added: "TX"
- board text added: "VBAT"
- board text added: "VCC"
- board text added: "VID_IN"
- board text added: "VID_OUT"

Commit message: layout progress
Parts:
- added TP37: sensors, Solderpoint:Solderpad, F.Cu at (124.3, 80.6)
- added TP38: sensors, Solderpoint:Solderpad, F.Cu at (126.7, 80.6)
- R28: moved to B.Cu
- TP33, TP34, TP35, TP36: value power -> sensors
- moved R21 19.6 mm to (122.1, 85.8), turned to 0 degrees
- moved TP4 19.4 mm to (128.1, 80.1), turned to 180 degrees
- moved C37 15.5 mm to (120.8, 87.1), turned to -90 degrees
- moved TP17 14.5 mm to (115.7, 93.0), turned to -90 degrees
- moved C55 14.0 mm to (140.2, 88.7), turned to 90 degrees
- moved J10 9.88 mm to (135.0, 80.5)
- moved R28 9.77 mm to (135.0, 85.2)
- moved U14 9.37 mm to (136.3, 88.7), turned to 180 degrees
- moved D8 9.12 mm to (131.3, 84.6)
- moved TP28 8.08 mm to (137.9, 80.3)
- moved C20 7.93 mm to (133.8, 94.2), turned to -90 degrees
- moved R22 7.60 mm to (128.6, 85.8)
- moved C10 7.58 mm to (143.9, 97.2)
- moved J4 7.29 mm to (126.5, 80.4)
- moved C16 7.09 mm to (147.1, 95.4), turned to 180 degrees
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Connections:
- J10 pad 1: +5V -> +3.3V
Routing:
- net /Power/D-: track 2.94 -> 0.00 mm
- net /Power/D+: track 2.94 -> 0.00 mm
- net unconnected-(U13-NC-Pad27): track 0.72 -> 0.00 mm
Other:
- board text added: "12V"
- board text added: "3.3V"
- board text added: "9V"
- board text added: "VTX_TX"

Commit message: hella shit configured, layout progress
Parts:
- added TP39: sensors, Solderpoint:Solderpad, F.Cu at (138.8, 114.5)
- added TP40: sensors, Solderpoint:Solderpad, F.Cu at (140.8, 114.5)
- added TP41: sensors, Solderpoint:Solderpad, F.Cu at (115.0, 92.5)
- added TP42: sensors, Solderpoint:Solderpad, F.Cu at (115.0, 90.5)
- added TP43: power, Solderpoint:Solderpad, F.Cu at (138.5, 111.6)
- added TP45: power, Solderpoint:Solderpad, F.Cu at (136.5, 111.6)
- C18, C20, D8, R28, U6: moved to F.Cu
- C8: footprint Capacitor_SMD:C_0603_1608Metric -> Capacitor_SMD:C_0402_1005Metric
- moved TP21 35.5 mm to (132.5, 113.6), turned to 180 degrees
- moved TP1 35.5 mm to (134.4, 113.6), turned to 180 degrees
- moved TP28 34.5 mm to (128.5, 113.5), turned to 180 degrees
- moved J2 29.8 mm to (132.7, 80.5), turned to 0 degrees
- moved TP25 28.9 mm to (130.5, 111.5), turned to 0 degrees
- moved J3 27.2 mm to (116.5, 89.5), turned to 90 degrees
- moved TP22 26.3 mm to (115.0, 86.5), turned to 90 degrees
- moved C53 26.3 mm to (142.4, 85.6), turned to 0 degrees
- moved C38 25.9 mm to (131.2, 83.5), turned to 90 degrees
- moved C19 25.5 mm to (119.5, 107.1), turned to 90 degrees
- moved C39 25.0 mm to (130.0, 84.0), turned to 90 degrees
- moved C36 25.0 mm to (129.1, 84.0), turned to 90 degrees
- moved C17 24.7 mm to (123.0, 109.7)
- moved R21 24.3 mm to (124.0, 110.0)
- moved C37 23.3 mm to (122.2, 110.4)
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Connections:
- net CANH renamed CAN_P
- net CANL renamed CAN_N
- C9 pad 1: +5V_USB -> +5V
- D1 pad 1: VBAT -> +VBAT
- J1 pad A4/B9: +5V_USB -> +5V
- J1 pad B4/A9: +5V_USB -> +5V
- J11 pad 2: EXPANSION_TX -> EXPANSION_RX
- J11 pad 3: EXPANSION_RX -> EXPANSION_TX
- J2 pad 1: +pwr_out -> GND
- J2 pad 4: GND -> +5V
- J4 pad 1: +5V -> GND
- J4 pad 6: GND -> +5V
- J6 pad 1: VBAT -> +VBAT
- Q1 pad 3: VBAT -> +VBAT
- R7 pad 2: VBAT -> +VBAT
- TP14 pad 1: +VABT -> +VBAT
- TP31 pad 1: +5V -> GND
- TP35 pad 1: GPS_SCL -> GPS_TX
- TP36 pad 1: GPS_SDA -> GPS_RX
- U10 pad 1: IMU2_MISO -> IMU_MISO
- U10 pad 12: IMU2_CS -> IMU_CS
- U10 pad 13: IMU2_SCLK -> IMU_SCLK
- U10 pad 14: IMU2_MOSI -> IMU_MOSI
- U10 pad 4: IMU2_INT1 -> IMU_INT1
- U2 pad 5: +5V_USB -> +5V
- U7 pad 2: OSD_CS -> unconnected-(U7-PE3-Pad2)
- U7 pad 24: GPS_TX -> VTX_TX
- U7 pad 25: GPS_RX -> unconnected-(U7-PA3-Pad25)
- U7 pad 28: IMU_CS -> FLASH_CS
- U7 pad 29: IMU_SCLK -> FLASH_SCLK
- U7 pad 3: unconnected-(U7-PE4-Pad3) -> IMU2_INT1
- U7 pad 30: IMU_MISO -> FLASH_MISO
- U7 pad 31: IMU_MOSI -> FLASH_MOSI
- U7 pad 32: IMU_INT1 -> unconnected-(U7-PC4-Pad32)
- U7 pad 51: EXPANSION_RX -> TELEMETRY_RX
- U7 pad 52: EXPANSION_TX -> TELEMETRY_TX
- U7 pad 53: WIFI/RC_TX -> EXPANSION_TX
- U7 pad 54: WIFI/RC_RX -> EXPANSION_RX
- U7 pad 55: TELEMETRY_TX -> WIFI/RC_TX
- U7 pad 56: TELEMETRY_RX -> WIFI/RC_RX
- U7 pad 7: unconnected-(U7-PC13-Pad7) -> OSD_CS
- U7 pad 78: IMU2_SCLK -> IMU_SCLK
- U7 pad 79: IMU2_MISO -> IMU_MISO
- U7 pad 80: IMU2_MOSI -> IMU_MOSI
- U7 pad 83: IMU2_INT1 -> IMU_INT1
- U7 pad 84: IMU2_CS -> IMU_CS
- U7 pad 88: FLASH_CS -> IMU2_CS
- U7 pad 89: FLASH_SCLK -> IMU2_SCLK
- U7 pad 90: FLASH_MISO -> IMU2_MISO
- U7 pad 91: FLASH_MOSI -> IMU2_MOSI
- U7 pad 97: unconnected-(U7-PE0-Pad97) -> GPS_RX
- U7 pad 98: VTX_TX -> GPS_TX
- U8 pad 1: IMU_MISO -> IMU2_MISO
- U8 pad 12: IMU_CS -> IMU2_CS
- U8 pad 13: IMU_SCLK -> IMU2_SCLK
- U8 pad 14: IMU_MOSI -> IMU2_MOSI
- U8 pad 4: IMU_INT1 -> IMU2_INT1
Routing:
- net +3.3V: track 0.00 -> 81.6 mm, vias 0 -> 16
- net OSD_CS: track 0.00 -> 25.3 mm, vias 0 -> 1
- net OSD_SCLK: track 0.00 -> 25.2 mm, vias 0 -> 1
- net OSD_MOSI: track 0.00 -> 24.5 mm, vias 0 -> 1
- net OSD_MISO: track 0.00 -> 22.0 mm, vias 0 -> 1
- net VBAT_Filtered: track 0.00 -> 17.2 mm
- net +5V: track 0.00 -> 17.2 mm, vias 0 -> 6
- net M8: track 0.00 -> 12.3 mm, vias 0 -> 1
- net +VBAT: track 0.00 -> 12.0 mm, vias 0 -> 5
- net M7: track 0.00 -> 10.7 mm, vias 0 -> 1
- net M6: track 0.00 -> 10.1 mm, vias 0 -> 1
- net M5: track 0.00 -> 9.80 mm, vias 0 -> 1
- net /Power/D-: track 0.00 -> 9.40 mm
- net ST_SWCLK: track 0.00 -> 9.19 mm, vias 0 -> 2
- net /Power/D+: track 0.00 -> 8.62 mm, vias 0 -> 2
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- added copper zone on In2.Cu, net +3.3V
- added copper zone on In2.Cu, net +5V
- added copper zone on B.Cu, net GND
- added copper zone on F.Cu, net GND
- added copper zone on In1.Cu, net GND
- added copper zone on In2.Cu, net GND
- added copper zone on In3.Cu, net GND
- added copper zone on In4.Cu, net GND
Other:
- board text added: "+5V"
- board text added: "CANH"
- board text added: "CANL"
- board text added: "GPS RX"
- board text added: "GPS TX"
- board text added: "M1"
- board text added: "M3"
- board text added: "M4"
- board text added: "PWR"
- board text added: "RX1"
- board text added: "S1"
- board text added: "S2"
- board text added: "S3"
- board text added: "S4"
- board text added: "SCL2"
- board text added: "SDA2"
- board text added: "STS1"
- board text added: "STS2"
- board text added: "TX1"
- board text added: "VIDEO OUT"
- board text added: "VTX TX"
