File: Hardware/connectors.kicad_sch (KiCad schematic)
At the start: 54 parts, among them J10 CAN BUS, J11 CAN BUS, J2 FPV, J3 ST_LINK, J4 GPS, J5 Airspeed sensor, J6 4in1 ESC, J7 RC Receiver, J8 VTX, J9 DJI

Commit message: added zener diode, more layout, Power verificatoin
Parts:
- removed TP25, TP28: power, Solderpoint:Solderpad, symbol Connector:TestPoint

Commit message: more routing and placement
Connections:
- net +pwr_out: no longer J5.1 (Pin_1)
- net I2C1_SCL: now also J5.3 (Pin_3); no longer J5.2 (Pin_2)
- net I2C1_SDA: now also J5.2 (Pin_2); no longer J5.3 (Pin_3)
- new net +3V3: J5.1 (Pin_1)
Changed lines of the file:
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@@
 		)
 	)
-	(global_label "I2C1_SCL"
+	(global_label "ST_SWCLK"
 		(shape input)
-		(at 198.12 147.32 180)
+		(at 293.37 62.23 180)
 		(fields_autoplaced yes)
 		(effects
 			(font
 				(size 0.762 0.762)
+				(thickness 0.1524)
+				(bold yes)
 			)
 			(justify right)
 		)
 		(property "Intersheetrefs" "${INTERSHEET_REFS}"
-			(at 191.0671 147.32 0)
+			(at 285.6687 62.23 0)
 			(effects
 				(font
@@
 		)
 	)
-	(global_label "ST_SWCLK"
+	(global_label "WIFI/RC_RX"
 		(shape input)
-		(at 293.37 62.23 180)
+		(at 234.95 60.96 180)
 		(fields_autoplaced yes)
 		(effects
@@
 		)
 		(property "Intersheetrefs" "${INTERSHEET_REFS}"
-			(at 285.6687 62.23 0)
+			(at 226.4141 60.96 0)
 			(effects
 				(font
@@
 		)
 	)
-	(global_label "WIFI/RC_RX"
+	(global_label "WIFI/RC_TX"
 		(shape input)
-		(at 234.95 60.96 180)
+		(at 234.95 58.42 180)
 		(fields_autoplaced yes)
 		(effects
@@
 		)
 		(property "Intersheetrefs" "${INTERSHEET_REFS}"
-			(at 226.4141 60.96 0)
+			(at 226.4141 58.42 0)
 			(effects
 				(font
@@
 		)
 	)
-	(global_label "WIFI/RC_TX"
+	(global_label "I2C1_SDA"
 		(shape input)
-		(at 234.95 58.42 180)
+		(at 198.12 147.32 180)
 		(fields_autoplaced yes)
 		(effects
 			(font
 				(size 0.762 0.762)
-				(thickness 0.1524)
-				(bold yes)
 			)
 			(justify right)
 		)
 		(property "Intersheetrefs" "${INTERSHEET_REFS}"
-			(at 226.4141 58.42 0)
+			(at 191.0309 147.32 0)
 			(effects
 				(font
@@
 		)
 	)
-	(global_label "DJI_TX"
+	(global_label "I2C1_SCL"
 		(shape input)
-		(at 257.81 147.32 180)
+		(at 198.12 149.86 180)
 		(fields_autoplaced yes)
 		(effects
 			(font
 				(size 0.762 0.762)
-				(thickness 0.1524)
-				(bold yes)
 			)
 			(justify right)
 		)
 		(property "Intersheetrefs" "${INTERSHEET_REFS}"
-			(at 251.9593 147.32 0)
+			(at 191.0671 149.86 0)
 			(effects
 				(font
@@
 		)
 	)
-	(global_label "S2"
+	(global_label "DJI_TX"
 		(shape input)
-		(at 77.47 168.91 270)
+		(at 257.81 147.32 180)
 		(fields_autoplaced yes)
 		(effects
@@
 		)
 		(property "Intersheetrefs" "${INTERSHEET_REFS}"
-			(at 77.47 175.9217 90)
+			(at 251.9593 147.32 0)
 			(effects
 				(font
@@
 		)
 	)
-	(global_label "CAN_N"
+	(global_label "S2"
 		(shape input)
-		(at 46.99 213.36 90)
+		(at 77.47 168.91 270)
 		(fields_autoplaced yes)
 		(effects
@@
 				(bold yes)
 			)
-			(justify left)
+			(justify right)
 		)
 		(property "Intersheetrefs" "${INTERSHEET_REFS}"
-			(at 46.99 208.4528 90)
+			(at 77.47 175.9217 90)
 			(effects
 				(font
 					(size 1.27 1.27)
 				)
-				(justify left)
+				(justify right)
 				(hide yes)
 			)
 		)
 	)
-	(global_label "CURR"
+	(global_label "CAN_N"
 		(shape input)
-		(at 289.56 101.6 0)
+		(at 46.99 213.36 90)
 		(fields_autoplaced yes)
 		(effects
@@
 		)
 		(property "Intersheetrefs" "${INTERSHEET_REFS}"
-			(at 294.7212 101.6 0)
+			(at 46.99 208.4528 90)
 			(effects
 				(font
@@
 		)
 	)
-	(global_label "I2C1_SDA"
+	(global_label "CURR"
 		(shape input)
-		(at 198.12 149.86 180)
+		(at 289.56 101.6 0)
 		(fields_autoplaced yes)
 		(effects
 			(font
 				(size 0.762 0.762)
+				(thickness 0.1524)
+				(bold yes)
 			)
-			(justify right)
+			(justify left)
 		)
 		(property "Intersheetrefs" "${INTERSHEET_REFS}"
-			(at 191.0309 149.86 0)
+			(at 294.7212 101.6 0)
 			(effects
 				(font
 					(size 1.27 1.27)
 				)
-				(justify right)
+				(justify left)
 				(hide yes)
 			)
@@
 		(on_board yes)
 		(dnp no)
-		(fields_autoplaced yes)
 		(property "Reference" "#PWR0141"
 			(at 196.85 144.78 0)
@@
 			)
 		)
-		(property "Value" "+pwr_out"
-			(at 196.85 135.89 0)
+		(property "Value" "+3V3"
+			(at 192.278 136.652 0)
 			(effects
 				(font
 					(size 1.27 1.27)
 				)
+				(justify left)
 			)
 		)

Commit message: First iteration layout done
Parts:
- removed TP11: power, Solderpoint:Solderpad, symbol Connector:TestPoint
- removed TP19: GND, Solderpoint:Solderpad, symbol Connector:TestPoint
- added TP25: power, Solderpoint:Solderpad, symbol Connector:TestPoint
- added TP28: sensors, Solderpoint:Solderpad, symbol Connector:TestPoint
Connections:
- net +3V3 is gone; now on net +3.3V: J5.1 (Pin_1)
- net +5V: now also TP25.1
- net CAN_N: no longer TP37.1
- net CAN_P: no longer TP38.1
- net GPS_SCL: now also TP37.1
- net GPS_SDA: now also TP38.1
- net VIDEO_IN: now also TP28.1
- net WIFI/RC_RX: now also J7.2 (Pin_2); no longer J7.3 (Pin_3)
- net WIFI/RC_TX: now also J7.3 (Pin_3); no longer J7.2 (Pin_2)
