File: Hardware/Sensors.kicad_sch (KiCad schematic)
At the start: 41 parts, among them U10 BMI270, U11 LIS3MDLTR, U12 BMP388, U13 AT7456E, U14 SN65HVD230, U8 ICM-42688-P, U9 W25Q128JVSIQ, Y2 27Mhz 20pF

Commit message: minor Updates
Parts:
- added R31, R32: 4.7k, Resistor_SMD:R_0402_1005Metric, symbol Device:R_Small
Connections:
- net +3.3V: now also R31.1, R32.1
- new net GPS_SCL: R31.2
- new net GPS_SDA: R32.2
